File: DSP_TU.kicad_sch (KiCad schematic)
At the start: 72 parts, among them J1 Conn_01x07_Male, J2 Conn_01x08_Male, J3 USB_B, J5 1757569, K1 G3VM-601BY, K2 G3VM-601BY, T1 TY-141P, T2 TY-145P, U1 PIC32MZ0512EFE064-I_PT, U2 TLV2780CDBVT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

Commit message: PCB Rev B, changing dimensions, adding test points, adding resistors in UART lines, and correcting display pinout. hh
Parts:
- added J4, J6, J7: Conn_01x08_Male, Connector_PinHeader_2.54mm:PinHeader_1x08_P2.54mm_Vertical, symbol Connector:Conn_01x08_Male
- added R18, R19, R21: 1k, Resistor_SMD:R_0603_1608Metric_Pad0.98x0.95mm_HandSolder, symbol Device:R
- added R20: 10k, Resistor_SMD:R_0603_1608Metric_Pad0.98x0.95mm_HandSolder, symbol Device:R
Connections:
- net +3V3: now also J1.7 (Pin_7), R20.2; no longer J1.1 (Pin_1)
- net GND: now also J1.6 (Pin_6), J4.8 (Pin_8), J6.8 (Pin_8), J7.8 (Pin_8), R21.1; no longer J1.2 (Pin_2)
- net IDLEn: now also R20.1, R21.2
- net LOOP_KEY: now also J6.1 (Pin_1)
- net LOOP_SENSE: now also J6.2 (Pin_2)
- net PTT: now also J6.6 (Pin_6)
- net U1CTSn: now also J7.3 (Pin_3), R18.2; no longer U3.2 (RTS#)
- net U1RTSn: now also J7.1 (Pin_1)
- net U1RX: now also J7.4 (Pin_4), R19.1; no longer U3.20 (TXD)
- net U1TX: now also J7.2 (Pin_2)
- net WIFI_CSn: now also J4.4 (Pin_4)
- net WIFI_EN: now also J4.7 (Pin_7)
- net WIFI_IRQn: now also J4.5 (Pin_5)
- net WIFI_MOSI: now also J4.1 (Pin_1)
- net WIFI_RESETn: now also J4.6 (Pin_6)
- net WIFI_SPI_CLK: now also J4.3 (Pin_3)
- net WIFI_MISO_TP: now reaches R16.1, U7.17 (SPI_MISO)
- net WIFI_MISO_TP: now also J4.2 (Pin_2)
- net at U1.46 (AERXD1/ETXD3/RPD0/RTCC/INT0/RD0): now also J1.1 (Pin_1); no longer J1.7 (Pin_7)
- net at U1.47 (SOSCI/RPC13/RC13): now also J1.2 (Pin_2); no longer J1.6 (Pin_6)
- net at U1.48 (SOSCO/RPC14/T1CK/RC14): now also J1.3 (Pin_3); no longer J1.5 (Pin_5)
- net at U1.50 (ETXERR/AETXEN/RPD2/SDA3/RD2): now also J1.5 (Pin_5); no longer J1.3 (Pin_3)
- net AFSK_OUT: now reaches C10.2, C9.1, U2.1 (OUT), U2.4 (IN-)
- net AFSK_OUT: now also J6.7 (Pin_7)
- net AFSK_OUT_ENn renamed AFSK_OUT_EN
- new net: R19.2, U3.20 (TXD)
- new net: R18.1, U3.2 (RTS#)
- no-connect marks 38 -> 44
Other:
- note added: "ADC reads board rev on power up. Pin then low during idle and high during DSP operations."
- note added: "Display 7 +3V3 6 GND 5 DIN 4 CLK 4 CSn 2 DC 1 RSTn"
- note added: "In FT_PROG, select Hardware Specific, select Battery Charge Detect. Check Battery Charge Enable and Force Power Enable. For CBUS Signals, change C3 to PWREN#. This will make output C3 go low when the host computer has enumerated this chip. Also, since we set "Force Power Enable", above, PWREN# will also go low when a dedicated charger is used to drive the system. See FTDI AN 175. Under USB Config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"
- note added: "SPI2, INT3"
- note removed: "Display 1 +3V3 2 GND 3 DIN 4 CLK 5 CSn 6 DC 7 RSTn"
- note removed: "Program U3 to put open drain PWRENn on CBUS3 and set MaxPower to 500mA."
- moved on the sheet: C20, C21, C22, J1, J2, J5, R12, R16, R17, R27, U7
